Commit message: Add files via upload

File: src/robot/robot1_description/urdf/car.xacro (robot description, xacro)
@@ -112,20 +112,20 @@
         <parent link="car_base"/>
         <child link="laser_1"/>
-        <origin rpy="0 0 ${PI/2}" xyz="-1.995  0.995 0.205"/>
+        <origin rpy="0 0 ${PI/2}" xyz="-1.99  0.99 0.205"/>
     </joint>
     <joint name="laser_joint_2" type="fixed">
         <parent link="car_base"/>
         <child link="laser_2"/>
-        <origin rpy="0 0 ${PI/2}" xyz="1.995  0.995 0.205"/>
+        <origin rpy="0 0 ${PI/2}" xyz="1.99  0.99 0.205"/>
     </joint>
     <joint name="laser_joint_3" type="fixed">
         <parent link="car_base"/>
         <child link="laser_3"/>
-        <origin rpy="0 0 ${-PI/2}" xyz="1.995  -0.995 0.205"/>
+        <origin rpy="0 0 ${-PI/2}" xyz="1.99  -0.99 0.205"/>
     </joint>
     <joint name="laser_joint_4" type="fixed">
         <parent link="car_base"/>
         <child link="laser_4"/>
-        <origin rpy="0 0 ${-PI/2}" xyz="-1.995  -0.995 0.205"/>
+        <origin rpy="0 0 ${-PI/2}" xyz="-1.99  -0.99 0.205"/>
     </joint>
     <xacro:wheel name="left_wheel_1"/>
